File: EECD_22_6_remote_control.kicad_pcb (KiCad board)
At the start: 2 copper layers, 27 parts

Commit message: Schematic refactor
- Divide the schematic into hierarchical sheets
- Fix ERCs
- Remove unused footprints
- Add SWD connector
- Add bypass capacitors
Parts:
- removed IC**: SON50P300X300X80-11N-D, models:SON50P300X300X80-11N-D
- removed REF** (x13): R_0201_0603Metric, Resistor_SMD:R_0201_0603Metric
- removed REF**: SW_CuK_JS202011CQN_DPDT_Straight, Button_Switch_THT:SW_CuK_JS202011CQN_DPDT_Straight
- removed REF** (x4): CP_Elec_3x5.3, Capacitor_SMD:CP_Elec_3x5.3
- removed REF** (x3): LED_Avago_PLCC4_3.2x2.8mm_CW, LED_SMD:LED_Avago_PLCC4_3.2x2.8mm_CW
- removed REF** (x2): XDCR_COM-09032, models:XDCR_COM-09032
- removed REF**: nRF24L01_Breakout, RF_Module:nRF24L01_Breakout
- removed REF**: L_6.3x6.3_H3, Inductor_SMD:L_6.3x6.3_H3
- removed REF**: LQFP-64_10x10mm_P0.5mm, Package_QFP:LQFP-64_10x10mm_P0.5mm

Commit message: Use proper footprints for custom symbols
Parts:
- added BT1: Li-Ion, Local_Library:BAT_BCAAAW, F.Cu at (98.7, 59.1)
- added C1: 22pF, Capacitor_SMD:C_0603_1608Metric, F.Cu at (84.9, 107.2)
- added C10: 10μF, Capacitor_SMD:CP_Elec_6.3x5.4, F.Cu at (76.2, 123.6)
- added C11: 10μF, Capacitor_Tantalum_SMD:CP_EIA-3216-10_Kemet-I, F.Cu at (162.9, 80.0)
- added C2: 22pF, Capacitor_SMD:C_0603_1608Metric, F.Cu at (96.9, 107.2)
- added C3: 100nF, Capacitor_SMD:C_0603_1608Metric, F.Cu at (88.9, 107.2)
- added C4: 100nF, Capacitor_SMD:C_0603_1608Metric, F.Cu at (100.9, 107.2)
- added C5: 100nF, Capacitor_SMD:C_0603_1608Metric, F.Cu at (101.0, 92.5)
- added C6: 100nF, Capacitor_SMD:C_0603_1608Metric, F.Cu at (92.9, 107.2)
- added C7: 100nF, Capacitor_SMD:C_0603_1608Metric, F.Cu at (76.9, 107.2)
- added C8: 1.5nF, Capacitor_SMD:C_0603_1608Metric, F.Cu at (79.6, 128.9)
- added C9: 22μF, Capacitor_SMD:CP_Elec_6.3x5.4, F.Cu at (88.8, 117.1)
- added D1: LED_RGBK, LED_SMD:LED_Avago_PLCC4_3.2x2.8mm_CW, F.Cu at (139.2, 115.2)
- added D2: LED_RGBK, LED_SMD:LED_Avago_PLCC4_3.2x2.8mm_CW, F.Cu at (133.1, 119.6)
- added D3: LED_RGBK, LED_SMD:LED_Avago_PLCC4_3.2x2.8mm_CW, F.Cu at (133.1, 115.2)
- added J1: SWD, Connector_PinHeader_2.54mm:PinHeader_2x03_P2.54mm_Vertical, F.Cu at (115.7, 93.0)
- added JOY1: COM-09032, Local_Library:XDCR_COM-09032, F.Cu at (142.1, 76.7)
- added JOY2: COM-09032, Local_Library:XDCR_COM-09032, F.Cu at (85.0, 92.0)
- added L1: 10μH, Inductor_SMD:L_Bourns-SRN4018, F.Cu at (84.6, 124.0)
- added R1: 10kΩ, Resistor_SMD:R_0603_1608Metric, F.Cu at (72.9, 107.2)
- added R10: 100Ω, Resistor_SMD:R_0603_1608Metric, F.Cu at (148.2, 114.3)
- added R11: 100Ω, Resistor_SMD:R_0603_1608Metric, F.Cu at (132.0, 123.0)
- added R12: 100Ω, Resistor_SMD:R_0603_1608Metric, F.Cu at (132.0, 128.0)
- added R13: 100Ω, Resistor_SMD:R_0603_1608Metric, F.Cu at (136.1, 125.5)
- added R14: 100Ω, Resistor_SMD:R_0603_1608Metric, F.Cu at (138.1, 118.7)
- added R15: 100Ω, Resistor_SMD:R_0603_1608Metric, F.Cu at (142.1, 118.7)
- added R2: 10kΩ, Resistor_SMD:R_0603_1608Metric, F.Cu at (80.9, 107.2)
- added R3: 340kΩ, Resistor_SMD:R_0603_1608Metric, F.Cu at (76.9, 133.0)
- added R4: 15kΩ, Resistor_SMD:R_0603_1608Metric, F.Cu at (72.9, 135.6)
- added R5: 60.4kΩ, Resistor_SMD:R_0603_1608Metric, F.Cu at (72.9, 133.0)
- added R6: 200kΩ, Resistor_SMD:R_0603_1608Metric, F.Cu at (96.2, 114.3)
- added R7: 180Ω, Resistor_SMD:R_0603_1608Metric, F.Cu at (144.2, 114.3)
- added R8: 180Ω, Resistor_SMD:R_0603_1608Metric, F.Cu at (132.0, 125.5)
- added R9: 180Ω, Resistor_SMD:R_0603_1608Metric, F.Cu at (136.1, 123.0)
- added SW1: SW_SPST, Button_Switch_SMD:SW_DIP_SPSTx01_Slide_9.78x4.72mm_W8.61mm_P2.54mm, F.Cu at (77.2, 116.3)
- added U1: STM32L4P5RET6, Package_QFP:LQFP-64_10x10mm_P0.5mm, F.Cu at (106.2, 84.1)
- added U2: LTC3440EMS, Local_Library:SOP50P490X110-10N, F.Cu at (74.2, 129.7)
- added U3: NRF24L01_Breakout, RF_Module:nRF24L01_Breakout, F.Cu at (162.3, 64.4)
- added Y1: 16MHz, Crystal:Crystal_SMD_3225-4Pin_3.2x2.5mm, F.Cu at (116.0, 79.1)
