File: communication.kicad_sch (KiCad schematic)
At the start: 2 parts, among them U3 NRF24L01_Breakout

Commit message: Improve DCDC converter diagram
Other:
- company: Authors: H. Fedarovich, I. Kajdan -> Authors: A. Kotkov, I. Kajdan
Changed lines of the file:
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@@
   (title_block
     (title "Communication")
-    (date "2022-12-23")
+    (date "2022-12-28")
     (rev "${REVISION}")
-    (company "Authors: H. Fedarovich, I. Kajdan")
+    (company "Authors: A. Kotkov, I. Kajdan")
     (comment 1 "Reviewer: A. Bondyra")
   )
@@
   (symbol (lib_id "power:+3.3V") (at 149.86 80.01 0) (unit 1)
     (in_bom yes) (on_board yes) (fields_autoplaced)
-    (property "Reference" "#PWR021" (id 0) (at 149.86 83.82 0)
+    (property "Reference" "#PWR022" (id 0) (at 149.86 83.82 0)
       (effects (font (size 1.27 1.27)) hide)
     )
@@
   (symbol (lib_id "power:+3.3V") (at 175.26 93.98 0) (unit 1)
     (in_bom yes) (on_board yes) (fields_autoplaced)
-    (property "Reference" "#PWR022" (id 0) (at 175.26 97.79 0)
+    (property "Reference" "#PWR023" (id 0) (at 175.26 97.79 0)
       (effects (font (size 1.27 1.27)) hide)
     )
@@
   (symbol (lib_id "power:GND") (at 149.86 115.57 0) (unit 1)
     (in_bom yes) (on_board yes) (fields_autoplaced)
-    (property "Reference" "#PWR024" (id 0) (at 149.86 121.92 0)
+    (property "Reference" "#PWR025" (id 0) (at 149.86 121.92 0)
       (effects (font (size 1.27 1.27)) hide)
     )
@@
   (symbol (lib_id "power:GND") (at 175.26 102.87 0) (unit 1)
     (in_bom yes) (on_board yes)
-    (property "Reference" "#PWR023" (id 0) (at 175.26 109.22 0)
+    (property "Reference" "#PWR024" (id 0) (at 175.26 109.22 0)
       (effects (font (size 1.27 1.27)) hide)
     )
