File: input.kicad_sch (KiCad schematic)
At the start: 8 parts, among them SW2 SW_Push, SW3 SW_Push, SW4 SW_Push, SW5 SW_Push

Commit message: Arrange footprints
Parts:
- RV1, RV2: footprint (none) -> Potentiometer_THT:Potentiometer_ACP_CA14V-15_Vertical
- SW2, SW3, SW4, SW5: footprint (none) -> Button_Switch_THT:SW_PUSH_6mm_H13mm
Changed lines of the file:
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@@
   (title_block
     (title "Input")
-    (date "2022-12-29")
+    (date "2022-12-30")
     (rev "${REVISION}")
     (company "Authors: A. Kotkov, I. Kajdan")
@@
   (symbol (lib_id "power:GND") (at 102.87 110.49 0) (unit 1)
     (in_bom yes) (on_board yes)
-    (property "Reference" "#PWR034" (id 0) (at 102.87 116.84 0)
+    (property "Reference" "#PWR038" (id 0) (at 102.87 116.84 0)
       (effects (font (size 1.27 1.27)) hide)
     )
@@
       (effects (font (size 1.27 1.27)) (justify right))
     )
-    (property "Footprint" "" (id 2) (at 261.62 106.68 0)
+    (property "Footprint" "Potentiometer_THT:Potentiometer_ACP_CA14V-15_Vertical" (id 2) (at 261.62 106.68 0)
       (effects (font (size 1.27 1.27)) hide)
     )
@@
       (effects (font (size 1.27 1.27)) (justify right))
     )
-    (property "Footprint" "" (id 2) (at 76.2 102.87 0)
+    (property "Footprint" "Button_Switch_THT:SW_PUSH_6mm_H13mm" (id 2) (at 76.2 102.87 0)
       (effects (font (size 1.27 1.27)) hide)
     )
@@
   (symbol (lib_id "power:+3.3V") (at 142.24 91.44 0) (unit 1)
     (in_bom yes) (on_board yes) (fields_autoplaced)
-    (property "Reference" "#PWR027" (id 0) (at 142.24 95.25 0)
+    (property "Reference" "#PWR031" (id 0) (at 142.24 95.25 0)
       (effects (font (size 1.27 1.27)) hide)
     )
@@
   (symbol (lib_id "power:GND") (at 143.51 120.65 0) (unit 1)
     (in_bom yes) (on_board yes)
-    (property "Reference" "#PWR037" (id 0) (at 143.51 127 0)
+    (property "Reference" "#PWR041" (id 0) (at 143.51 127 0)
       (effects (font (size 1.27 1.27)) hide)
     )
@@
   (symbol (lib_id "power:+3.3V") (at 182.88 91.44 0) (unit 1)
     (in_bom yes) (on_board yes) (fields_autoplaced)
-    (property "Reference" "#PWR028" (id 0) (at 182.88 95.25 0)
+    (property "Reference" "#PWR032" (id 0) (at 182.88 95.25 0)
       (effects (font (size 1.27 1.27)) hide)
     )
@@
   (symbol (lib_id "power:GND") (at 261.62 111.76 0) (unit 1)
     (in_bom yes) (on_board yes)
-    (property "Reference" "#PWR036" (id 0) (at 261.62 118.11 0)
+    (property "Reference" "#PWR040" (id 0) (at 261.62 118.11 0)
       (effects (font (size 1.27 1.27)) hide)
     )
@@
   (symbol (lib_id "power:GND") (at 38.1 110.49 0) (unit 1)
     (in_bom yes) (on_board yes)
-    (property "Reference" "#PWR031" (id 0) (at 38.1 116.84 0)
+    (property "Reference" "#PWR035" (id 0) (at 38.1 116.84 0)
       (effects (font (size 1.27 1.27)) hide)
     )
@@
   (symbol (lib_id "power:GND") (at 184.15 120.65 0) (unit 1)
     (in_bom yes) (on_board yes)
-    (property "Reference" "#PWR038" (id 0) (at 184.15 127 0)
+    (property "Reference" "#PWR042" (id 0) (at 184.15 127 0)
       (effects (font (size 1.27 1.27)) hide)
     )
@@
       (effects (font (size 1.27 1.27)) (justify right))
     )
-    (property "Footprint" "" (id 2) (at 97.79 102.87 0)
+    (property "Footprint" "Button_Switch_THT:SW_PUSH_6mm_H13mm" (id 2) (at 97.79 102.87 0)
       (effects (font (size 1.27 1.27)) hide)
     )
@@
   (symbol (lib_id "power:GND") (at 81.28 110.49 0) (unit 1)
     (in_bom yes) (on_board yes)
-    (property "Reference" "#PWR033" (id 0) (at 81.28 116.84 0)
+    (property "Reference" "#PWR037" (id 0) (at 81.28 116.84 0)
       (effects (font (size 1.27 1.27)) hide)
     )
@@
       (effects (font (size 1.27 1.27)) (justify right))
     )
-    (property "Footprint" "" (id 2) (at 33.02 102.87 0)
+    (property "Footprint" "Button_Switch_THT:SW_PUSH_6mm_H13mm" (id 2) (at 33.02 102.87 0)
       (effects (font (size 1.27 1.27)) hide)
     )
@@
       (effects (font (size 1.27 1.27)) (justify right))
     )
-    (property "Footprint" "" (id 2) (at 233.68 106.68 0)
+    (property "Footprint" "Potentiometer_THT:Potentiometer_ACP_CA14V-15_Vertical" (id 2) (at 233.68 106.68 0)
       (effects (font (size 1.27 1.27)) hide)
     )
@@
   (symbol (lib_id "power:+3.3V") (at 261.62 101.6 0) (unit 1)
     (in_bom yes) (on_board yes) (fields_autoplaced)
-    (property "Reference" "#PWR030" (id 0) (at 261.62 105.41 0)
+    (property "Reference" "#PWR034" (id 0) (at 261.62 105.41 0)
       (effects (font (size 1.27 1.27)) hide)
     )
@@
   (symbol (lib_id "power:GND") (at 233.68 111.76 0) (unit 1)
     (in_bom yes) (on_board yes)
-    (property "Reference" "#PWR035" (id 0) (at 233.68 118.11 0)
+    (property "Reference" "#PWR039" (id 0) (at 233.68 118.11 0)
       (effects (font (size 1.27 1.27)) hide)
     )
@@
       (effects (font (size 1.27 1.27)) (justify right))
     )
-    (property "Footprint" "" (id 2) (at 54.61 102.87 0)
+    (property "Footprint" "Button_Switch_THT:SW_PUSH_6mm_H13mm" (id 2) (at 54.61 102.87 0)
       (effects (font (size 1.27 1.27)) hide)
     )
@@
   (symbol (lib_id "power:GND") (at 59.69 110.49 0) (unit 1)
     (in_bom yes) (on_board yes)
-    (property "Reference" "#PWR032" (id 0) (at 59.69 116.84 0)
+    (property "Reference" "#PWR036" (id 0) (at 59.69 116.84 0)
       (effects (font (size 1.27 1.27)) hide)
     )
@@
   (symbol (lib_id "power:+3.3V") (at 233.68 101.6 0) (unit 1)
     (in_bom yes) (on_board yes) (fields_autoplaced)
-    (property "Reference" "#PWR029" (id 0) (at 233.68 105.41 0)
-      (effects (font (size 1.27 1.27)) hide)
-    )
+    (property "Reference" "#PWR033" (id 0) (at 233.68 105.41 0)
+      (effects (font (size 1.27 1.27)) hide)
+    )

Commit message: Use more appropriate MCU pins for peripherals
Parts:
- renumbered RV2 to RV1, RV1 to RV2
Connections:
- net GND: now also SW2.2, SW3.2, SW4.2, SW5.2; no longer SW2.1, SW3.1, SW4.1, SW5.1
- net POT1: now also RV1.2; no longer RV2.2
- net POT2: now also RV2.2; no longer RV1.2
- net SW1: now also SW2.1; no longer SW2.2
- net SW2: now also SW3.1; no longer SW3.2
- net SW3: now also SW4.1; no longer SW4.2
- net SW4: now also SW5.1; no longer SW5.2
Other:
- moved on the sheet: RV1, RV2
Changed lines of the file:
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@@
     (pin "1")
   )
-  (symbol (lib_id "Device:R_Potentiometer_Small") (at 261.62 106.68 0) (mirror y) (unit 1)
-    (in_bom yes) (on_board yes)
-    (property "Reference" "RV2" (id 0) (at 264.16 105.4099 0)
-      (effects (font (size 1.27 1.27)) (justify right))
-    )
-    (property "Value" "100kΩ" (id 1) (at 264.16 107.9499 0)
-      (effects (font (size 1.27 1.27)) (justify right))
-    )
-    (property "Footprint" "Potentiometer_THT:Potentiometer_ACP_CA14V-15_Vertical" (id 2) (at 261.62 106.68 0)
-      (effects (font (size 1.27 1.27)) hide)
-    )
-    (property "Datasheet" "~" (id 3) (at 261.62 106.68 0)
-      (effects (font (size 1.27 1.27)) hide)
-    )
-    (pin "1")
-    (pin "2")
-    (pin "3")
-  )
-  (symbol (lib_id "Switch:SW_Push") (at 81.28 102.87 90) (unit 1)
+  (symbol (lib_id "Device:R_Potentiometer_Small") (at 233.68 106.68 0) (mirror y) (unit 1)
+    (in_bom yes) (on_board yes)
+    (property "Reference" "RV1" (id 0) (at 236.22 105.4099 0)
+      (effects (font (size 1.27 1.27)) (justify right))
+    )
+    (property "Value" "100kΩ" (id 1) (at 236.22 107.9499 0)
+      (effects (font (size 1.27 1.27)) (justify right))
+    )
+    (property "Footprint" "Potentiometer_THT:Potentiometer_ACP_CA14V-15_Vertical" (id 2) (at 233.68 106.68 0)
+      (effects (font (size 1.27 1.27)) hide)
+    )
+    (property "Datasheet" "~" (id 3) (at 233.68 106.68 0)
+      (effects (font (size 1.27 1.27)) hide)
+    )
+    (pin "1")
+    (pin "2")
+    (pin "3")
+  )
+  (symbol (lib_id "Switch:SW_Push") (at 81.28 102.87 90) (mirror x) (unit 1)
     (in_bom yes) (on_board yes) (fields_autoplaced)
     (property "Reference" "SW4" (id 0) (at 82.55 101.5999 90)
@@
     (pin "1")
   )
-  (symbol (lib_id "Switch:SW_Push") (at 102.87 102.87 90) (unit 1)
+  (symbol (lib_id "Switch:SW_Push") (at 102.87 102.87 90) (mirror x) (unit 1)
     (in_bom yes) (on_board yes) (fields_autoplaced)
     (property "Reference" "SW5" (id 0) (at 104.14 101.5999 90)
@@
     (pin "1")
   )
-  (symbol (lib_id "Switch:SW_Push") (at 38.1 102.87 90) (unit 1)
+  (symbol (lib_id "Switch:SW_Push") (at 38.1 102.87 90) (mirror x) (unit 1)
     (in_bom yes) (on_board yes) (fields_autoplaced)
     (property "Reference" "SW2" (id 0) (at 39.37 101.5999 90)
@@
     (pin "9")
   )
-  (symbol (lib_id "Device:R_Potentiometer_Small") (at 233.68 106.68 0) (mirror y) (unit 1)
-    (in_bom yes) (on_board yes) (fields_autoplaced)
-    (property "Reference" "RV1" (id 0) (at 236.22 105.4099 0)
-      (effects (font (size 1.27 1.27)) (justify right))
-    )
-    (property "Value" "100kΩ" (id 1) (at 236.22 107.9499 0)
-      (effects (font (size 1.27 1.27)) (justify right))
-    )
-    (property "Footprint" "Potentiometer_THT:Potentiometer_ACP_CA14V-15_Vertical" (id 2) (at 233.68 106.68 0)
-      (effects (font (size 1.27 1.27)) hide)
-    )
-    (property "Datasheet" "~" (id 3) (at 233.68 106.68 0)
+  (symbol (lib_id "Device:R_Potentiometer_Small") (at 261.62 106.68 0) (mirror y) (unit 1)
+    (in_bom yes) (on_board yes) (fields_autoplaced)
+    (property "Reference" "RV2" (id 0) (at 264.16 105.4099 0)
+      (effects (font (size 1.27 1.27)) (justify right))
+    )
+    (property "Value" "100kΩ" (id 1) (at 264.16 107.9499 0)
+      (effects (font (size 1.27 1.27)) (justify right))
+    )
+    (property "Footprint" "Potentiometer_THT:Potentiometer_ACP_CA14V-15_Vertical" (id 2) (at 261.62 106.68 0)
+      (effects (font (size 1.27 1.27)) hide)
+    )
+    (property "Datasheet" "~" (id 3) (at 261.62 106.68 0)
       (effects (font (size 1.27 1.27)) hide)
     )
@@
     (pin "1")
   )
-  (symbol (lib_id "Switch:SW_Push") (at 59.69 102.87 90) (unit 1)
+  (symbol (lib_id "Switch:SW_Push") (at 59.69 102.87 90) (mirror x) (unit 1)
     (in_bom yes) (on_board yes) (fields_autoplaced)
     (property "Reference" "SW3" (id 0) (at 60.96 101.5999 90)
